Commit message: 命名调整

File: model/xh_urdf/urdf/xh.urdf (robot description, URDF)
Before this commit: robot xh_urdf, 17 links, 16 joints
Links:
- link FL_foot: mass 0.00751392687794971 -> 0.03; geometry collision sphere radius=0.03; visual mesh filename=package://xh_urdf/meshes/FL_foot.STL
- link FR_foot: mass 0.00751392769459795 -> 0.03; geometry collision sphere radius=0.03; visual mesh filename=package://xh_urdf/meshes/FR_foot.STL
- link RL_foot: mass 0.00751392725509898 -> 0.03; geometry collision sphere radius=0.03; visual mesh filename=package://xh_urdf/meshes/RL_foot.STL
- link RR_foot: mass 0.00751426922402197 -> 0.03; geometry collision sphere radius=0.03; visual mesh filename=package://xh_urdf/meshes/RR_foot.STL
